File: OpenRX-Mono/OpenRX-Mono.kicad_pcb (KiCad board)
At the start: 6 copper layers, 10 x 16.3 mm, 61 parts, among them J1 Conn_Coaxial_Small, T1 0900PC16J0042001E, U1 ESP32-C3, U2 TLV75533PDQNR, U3 LR1121IMLTRT, U4 RFX2401C, U5 SKY13373-460LF, X1 CJ17-400001010B20

Commit message: OpenRX-Mono: PCB doc properties, 3D model fixes, target update, renders
Board file gains DOC_* properties and corrected 3D model references
(RFX2401C EP1.7, QFN-12 BL). ELRS target: corrected LR1121 RF switch
control table, enable radio DCDC, WS2812 RGB LED instead of plain LED.
Re-rendered README images.

Co-Authored-By: Claude Fable 5 <noreply@anthropic.com>
Routing:
- net GND: track 14.3 -> 7.80 mm, vias 66 -> 63
