File: OpenRX-Mono/OpenRX-Mono.kicad_pcb (KiCad board)
At the start: 6 copper layers, 10 x 16.3 mm, 61 parts, among them J1 Conn_Coaxial_Small, T1 0900PC16J0042001E, U1 ESP32-C3, U2 TLV75533PDQNR, U3 LR1121IMLTRT, U4 RFX2401C, U5 SKY13373-460LF, X1 CJ17-400001010B20

Commit message: changed 3.3V supply on clocks, added text, enlarged pads
Parts:
- moved TP1 1.00 mm to (101.2, 117.3)
- moved TP2 1.00 mm to (103.7, 117.3)
- moved TP3 1.00 mm to (106.3, 117.3)
- moved TP4 1.00 mm to (108.8, 117.3)
Connections:
- C13 pad 2: Net-(OSC1-VDD) -> +3V3
- OSC1 pad 4: Net-(OSC1-VDD) -> +3V3
- U3 pad 3: Net-(OSC1-VDD) -> unconnected-(U3-VTCXO-Pad3)
Routing:
- net Net-(OSC1-VDD): track 6.98 -> 0.00 mm
- net +3V3: track 14.0 -> 16.8 mm
Other:
- board size 10 x 16.3 mm -> 10 x 17.3 mm
