File: OpenRX-Mono/OpenRX-Mono.kicad_pcb (KiCad board)
At the start: 6 copper layers, 10 x 17.3 mm, 61 parts, among them J1 Conn_Coaxial_Small, T1 0900PC16J0042001E, U1 ESP32-C3, U2 TLV75533PDQNR, U3 LR1121IMLTRT, U4 RFX2401C, U5 SKY13373-460LF, X1 CJ17-400001010B20

Commit message: Rev 2 board work: routing optimisations, logo placement, 3D model fixes
Routing reworked on Lite (segments 313 to 256, vias 60 to 89), Lite-UFL
(317 to 269, 61 to 85) and Gemini (682 to 688, 196 to 243). ExpressLRS logo
placed on Mono.

3D model fixes on Gemini and Mono:

- RFX2401C (U4, U7) pointed at QFN-16_L3.0-W3.0-H0.9-P0.50.wrl with an offset
  of (-951.61, 821.31, 0), so the body rendered about a metre off the board and
  the land looked bare in the viewer. Repointed at the RFX2401C model that
  OpenRX-Shared.pretty/QFN-16_L3.0-W3.0-P0.50-BL-EP1.7.kicad_mod specifies,
  offset zeroed, 270 degree rotation kept.
- SKY13373 (U5, U8) carried no model reference at all. Added, matching the
  library footprint.

The boards now agree with the shared library on both, so Update Footprints from
Library preserves this rather than reverting it.

DRC reviewed: zero unconnected items on all four boards. The remaining items
are pre-existing and understood. The shorting_items reports on Lite and
Lite-UFL are all netted-copper against unnetted copper inside the multi-hole
TP footprints, never signal to signal, and are present at the previous commit
too. The copper_edge_clearance reports are the TP1-TP4 castellated pads sitting
on the board edge by design.

Co-Authored-By: Claude Opus 5 (1M context) <noreply@anthropic.com>
Parts:
- added G***: LOGO, OpenRX-Shared:expresslrs_logo, F.Cu at (101.8, 105.1)
Routing:
- net GND: vias 66 -> 78
