File: OpenRX-Mono/esp32c3_lr1121_mono.kicad_sch (KiCad schematic)
At the start: 61 parts, among them J1 Conn_Coaxial_Small, T1 0900PC16J0042001E, U1 ESP32-C3, U2 TLV75533PDQNR, U3 LR1121IMLTRT, U4 RFX2401C, U5 SKY13373-460LF, X1 CJ17-400001010B20

Commit message: sch: standardise LCSC/Manufacturer/MPN fields across all variants
Migrated LCSC part numbers out of variant-specific LCSC_Part fields into
the standard LCSC field, and backfilled Manufacturer/MPN from the LCSC
catalogue, on all four board variants (Gemini, Lite, Lite-UFL, Mono) and
the shared ESP32-C3/SX1281 RX core sheet.

kicad-skip reflowed each file on save, so the diffs are large but purely
formatting; a structural S-expression diff and ERC re-run on all 12
affected schematics (including the 4 unmodified top-level sheets) confirm
only property values changed, no nets/placement/footprints touched.

Known gap: L2/L3 in OpenRX-Gemini/esp32c3_lr1121_gemini.kicad_sch carry
LCSC C1035, which no longer resolves in the LCSC catalogue, so they have
no Manufacturer/MPN. Universal BOM lines for those parts will be
incomplete until a replacement part is sourced.

Co-Authored-By: Claude Fable 5 <noreply@anthropic.com>
Parts:
- AE1: MPN (none) -> 2450AT18A100E; Manufacturer (none) -> Johanson Dielectrics
- C1, C3: MPN (none) -> GRM0335C1H150JA01D; Manufacturer (none) -> muRata
- C10, C17, C25, C27, C28, C31, C4: MPN (none) -> GRM033R61A105ME44D; Manufacturer (none) -> muRata
- C11: MPN (none) -> GRM155R60J106ME44D; Manufacturer (none) -> muRata
- C12, C13, C14, C16, C5, C6, C9: MPN (none) -> GRM033R61E104KE14D; Manufacturer (none) -> muRata
- C15, C2, C23, C24: MPN (none) -> GRM0335C1H470JA01D; Manufacturer (none) -> muRata
- C18, C8: MPN (none) -> CL05A106MQ5NUNC; Manufacturer (none) -> Samsung Electro-Mechanics
- C19: MPN (none) -> GRM033R71E222KA12D; Manufacturer (none) -> muRata
- C20: MPN (none) -> GRM033R60J474KE90D; Manufacturer (none) -> muRata
- C21: MPN (none) -> GRM0335C1E221JA01D; Manufacturer (none) -> muRata
- C22: MPN (none) -> GRM033R71H102KA12D; Manufacturer (none) -> muRata
- C26: MPN (none) -> GRM033R61A103KA01J; Manufacturer (none) -> muRata
- C29, C30: MPN (none) -> GRM0335C1H1R2BA01D; Manufacturer (none) -> muRata
- C7: MPN (none) -> GRM0335C1H100FA01D; Manufacturer (none) -> muRata
- D1: LCSC (none) -> C5349953; LCSC Part C5349953 -> (none); MPN (none) -> XL-1010RGBC-2812B; Manufacturer (none) -> XINGLIGHT
- FL1: LCSC (none) -> C2651081; LCSC Part C2651081 -> (none)
- J1: MPN (none) -> U.FL-R-SMT-1(80); Manufacturer (none) -> HRS
- L1: MPN (none) -> MLZ1608N100LT000; Manufacturer (none) -> TDK
- L2: MPN (none) -> LQP03TN24NH02D; Manufacturer (none) -> muRata
- L3: MPN (none) -> LQP03TN2N0B02D; Manufacturer (none) -> muRata
- L4: MPN (none) -> LQP03TN2N5C02D; Manufacturer (none) -> muRata
- L5: MPN (none) -> LQW15AN47NJ00D; Manufacturer (none) -> muRata
- OSC1: LCSC (none) -> C22381772; LCSC Part C22381772 -> (none); MPN (none) -> OW7EL89CENUYO3YLC-32M; Manufacturer (none) -> YXC Crystal Oscillators
- R1: MPN (none) -> RC0201FR-07200RL; Manufacturer (none) -> YAGEO
- R2, R3, R4, R5: MPN (none) -> RC0201FR-0710KL; Manufacturer (none) -> YAGEO
- R6: MPN (none) -> ERJ-1GNF2200C; Manufacturer (none) -> PANASONIC
- R7, R8: MPN (none) -> RC0201FR-07100KL; Manufacturer (none) -> YAGEO
- T1: LCSC (none) -> C19842466; LCSC Part C19842466 -> (none); MPN (none) -> 0900PC16J0042001E; Manufacturer (none) -> Johanson Dielectrics
- U2: MPN (none) -> TLV75533PDQNR; Manufacturer (none) -> TI
- U3: LCSC (none) -> C7498014; LCSC Part C7498014 -> (none); MPN (none) -> LR1121IMLTRT; Manufacturer (none) -> SEMTECH
- U4: LCSC (none) -> C19213; LCSC Part C19213 -> (none); MPN (none) -> RFX2401C; Manufacturer (none) -> SKYWORKS
- X1: MPN (none) -> CJ17-400001010B20; Manufacturer (none) -> JSCJ
