File: OpenRX-Gemini/OpenRX-Gemini.kicad_pcb (KiCad board)
At the start: 6 copper layers, 17 x 15.7 mm, 85 parts, among them J1 Conn_Coaxial_Small, J2 Conn_Coaxial_Small, T1 0900PC16J0042001E, T2 0900PC16J0042001E, U1 ESP32-C3, U2 TLV75533PDQNR, U3 LR1121IMLTRT, U4 RFX2401C, U5 SKY13373-460LF, U6 LR1121IMLTRT, U7 RFX2401C, U8 SKY13373-460LF, U9 TS2306A 240GF MSM 9_C2976675, X1 CJ17-400001010B20

Commit message: changed 3.3V supply on clocks, added text, enlarged pads
Parts:
- added TP5: TestPoint, TestPoint:TestPoint_Pad_D1.5mm, F.Cu at (101.1, 102.3)
Connections:
- C13 pad 2: /Clock/VTCXO -> +3V3
- OSC1 pad 4: /Clock/VTCXO -> +3V3
- U3 pad 3: /LR1121_A/VTCXO -> unconnected-(U3-VTCXO-Pad3)
- U6 pad 3: /Clock/VTCXO -> unconnected-(U6-VTCXO-Pad3)
Routing:
- net /ESP32-C3/BOOT: track 14.8 -> 35.7 mm, vias 2 -> 3
- net /Clock/VTCXO: track 2.80 -> 0.00 mm
- net +3V3: track 28.9 -> 31.5 mm
Other:
- board text added: "BOOT"
- board text added: "OPEN"
