File: OpenRX-Gemini/clock.kicad_sch (KiCad schematic)
At the start: 2 parts

Commit message: sch: standardise LCSC/Manufacturer/MPN fields across all variants
Migrated LCSC part numbers out of variant-specific LCSC_Part fields into
the standard LCSC field, and backfilled Manufacturer/MPN from the LCSC
catalogue, on all four board variants (Gemini, Lite, Lite-UFL, Mono) and
the shared ESP32-C3/SX1281 RX core sheet.

kicad-skip reflowed each file on save, so the diffs are large but purely
formatting; a structural S-expression diff and ERC re-run on all 12
affected schematics (including the 4 unmodified top-level sheets) confirm
only property values changed, no nets/placement/footprints touched.

Known gap: L2/L3 in OpenRX-Gemini/esp32c3_lr1121_gemini.kicad_sch carry
LCSC C1035, which no longer resolves in the LCSC catalogue, so they have
no Manufacturer/MPN. Universal BOM lines for those parts will be
incomplete until a replacement part is sourced.

Co-Authored-By: Claude Fable 5 <noreply@anthropic.com>
Parts:
- C13: MPN (none) -> GRM033R61E104KE14D; Manufacturer (none) -> muRata
- OSC1: LCSC (none) -> C22381772; LCSC Part C22381772 -> (none); MPN (none) -> OW7EL89CENUYO3YLC-32M; Manufacturer (none) -> YXC Crystal Oscillators
