File: OpenRX-Gemini/esp32-c3.kicad_sch (KiCad schematic)
At the start: 36 parts, among them U1 ESP32-C3, U2 TLV75533PDQNR, U9 TS2306A 240GF MSM 9_C2976675, X1 CJ17-400001010B20

Commit message: sch: standardise LCSC/Manufacturer/MPN fields across all variants
Migrated LCSC part numbers out of variant-specific LCSC_Part fields into
the standard LCSC field, and backfilled Manufacturer/MPN from the LCSC
catalogue, on all four board variants (Gemini, Lite, Lite-UFL, Mono) and
the shared ESP32-C3/SX1281 RX core sheet.

kicad-skip reflowed each file on save, so the diffs are large but purely
formatting; a structural S-expression diff and ERC re-run on all 12
affected schematics (including the 4 unmodified top-level sheets) confirm
only property values changed, no nets/placement/footprints touched.

Known gap: L2/L3 in OpenRX-Gemini/esp32c3_lr1121_gemini.kicad_sch carry
LCSC C1035, which no longer resolves in the LCSC catalogue, so they have
no Manufacturer/MPN. Universal BOM lines for those parts will be
incomplete until a replacement part is sourced.

Co-Authored-By: Claude Fable 5 <noreply@anthropic.com>
Parts:
- AE1: MPN (none) -> 2450AT18A100E; Manufacturer (none) -> Johanson Dielectrics
- C1, C3: MPN (none) -> GRM0335C1H150JA01D; Manufacturer (none) -> muRata
- C10, C17, C25, C27, C28, C4: MPN (none) -> GRM033R61A105ME44D; Manufacturer (none) -> muRata
- C11: MPN (none) -> GRM155R60J106ME44D; Manufacturer (none) -> muRata
- C12, C5, C6, C9: MPN (none) -> GRM033R61E104KE14D; Manufacturer (none) -> muRata
- C18, C8: MPN (none) -> CL05A106MQ5NUNC; Manufacturer (none) -> Samsung Electro-Mechanics
- C26: MPN (none) -> GRM033R61A103KA01J; Manufacturer (none) -> muRata
- C29, C30: MPN (none) -> GRM0335C1H1R2BA01D; Manufacturer (none) -> muRata
- D1: LCSC (none) -> C5349953; LCSC Part C5349953 -> (none); MPN (none) -> XL-1010RGBC-2812B; Manufacturer (none) -> XINGLIGHT
- L2: MPN (none) -> LQP03TN24NH02D; Manufacturer (none) -> muRata
- L3: MPN (none) -> LQP03TN2N0B02D; Manufacturer (none) -> muRata
- L4: MPN (none) -> LQP03TN2N5C02D; Manufacturer (none) -> muRata
- R2, R3, R4, R5: MPN (none) -> RC0201FR-0710KL; Manufacturer (none) -> YAGEO
- U2: MPN (none) -> TLV75533PDQNR; Manufacturer (none) -> TI
- U9: LCSC (none) -> C2976675; LCSC Part C2976675 -> (none); MPN (none) -> TS2306A 240gf MSM 9; Manufacturer (none) -> SHOU HAN
- X1: MPN (none) -> CJ17-400001010B20; Manufacturer (none) -> JSCJ
