File: OpenRX-Gemini/lr1121.kicad_sch (KiCad schematic)
At the start: 24 parts, among them J1 Conn_Coaxial_Small, T1 0900PC16J0042001E, U3 LR1121IMLTRT, U4 RFX2401C, U5 SKY13373-460LF

Commit message: changed 3.3V supply on clocks, added text, enlarged pads
Connections:
- net VTCXO: no longer names the net of U3.3 (VTCXO)
- no-connect marks 11 -> 12
Changed lines of the file:
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@@
+	)
+	(no_connect
+		(at 114.3 119.38)
 	)
 	(no_connect
@@
 		(effects
 			(font
-				(size 1.27 1.27)
-			)
-			(justify right)
-		)
-	)
-	(hierarchical_label "VTCXO"
-		(shape output)
-		(at 114.3 119.38 180)
-		(effects
-			(font
