File: OpenRX-Gemini/lr1121.kicad_sch (KiCad schematic)
At the start: 24 parts, among them J1 Conn_Coaxial_Small, T1 0900PC16J0042001E, U3 LR1121IMLTRT, U4 RFX2401C, U5 SKY13373-460LF

Commit message: sch: standardise LCSC/Manufacturer/MPN fields across all variants
Migrated LCSC part numbers out of variant-specific LCSC_Part fields into
the standard LCSC field, and backfilled Manufacturer/MPN from the LCSC
catalogue, on all four board variants (Gemini, Lite, Lite-UFL, Mono) and
the shared ESP32-C3/SX1281 RX core sheet.

kicad-skip reflowed each file on save, so the diffs are large but purely
formatting; a structural S-expression diff and ERC re-run on all 12
affected schematics (including the 4 unmodified top-level sheets) confirm
only property values changed, no nets/placement/footprints touched.

Known gap: L2/L3 in OpenRX-Gemini/esp32c3_lr1121_gemini.kicad_sch carry
LCSC C1035, which no longer resolves in the LCSC catalogue, so they have
no Manufacturer/MPN. Universal BOM lines for those parts will be
incomplete until a replacement part is sourced.

Co-Authored-By: Claude Fable 5 <noreply@anthropic.com>
Parts:
- C14, C16: MPN (none) -> GRM033R61E104KE14D; Manufacturer (none) -> muRata
- C15, C2, C23, C24: MPN (none) -> GRM0335C1H470JA01D; Manufacturer (none) -> muRata
- C19: MPN (none) -> GRM033R71E222KA12D; Manufacturer (none) -> muRata
- C20: MPN (none) -> GRM033R60J474KE90D; Manufacturer (none) -> muRata
- C21: MPN (none) -> GRM0335C1E221JA01D; Manufacturer (none) -> muRata
- C22: MPN (none) -> GRM033R71H102KA12D; Manufacturer (none) -> muRata
- C31: MPN (none) -> GRM033R61A105ME44D; Manufacturer (none) -> muRata
- C7: MPN (none) -> GRM0335C1H100FA01D; Manufacturer (none) -> muRata
- FL1: LCSC (none) -> C2651081; LCSC Part C2651081 -> (none)
- J1: MPN (none) -> U.FL-R-SMT-1(80); Manufacturer (none) -> HRS
- L1: MPN (none) -> MLZ1608N100LT000; Manufacturer (none) -> TDK
- L5: MPN (none) -> LQW15AN47NJ00D; Manufacturer (none) -> muRata
- R1: MPN (none) -> RC0201FR-07200RL; Manufacturer (none) -> YAGEO
- R6: MPN (none) -> ERJ-1GNF2200C; Manufacturer (none) -> PANASONIC
- R7, R8: MPN (none) -> RC0201FR-07100KL; Manufacturer (none) -> YAGEO
- T1: LCSC (none) -> C19842466; LCSC Part C19842466 -> (none); MPN (none) -> 0900PC16J0042001E; Manufacturer (none) -> Johanson Dielectrics
- U3: LCSC (none) -> C7498014; LCSC Part C7498014 -> (none); MPN (none) -> LR1121IMLTRT; Manufacturer (none) -> SEMTECH
- U4: LCSC (none) -> C19213; LCSC Part C19213 -> (none); MPN (none) -> RFX2401C; Manufacturer (none) -> SKYWORKS
