File: OpenRX-Gemini/OpenRX-all.kicad_pcb (KiCad board)
At the start: 6 copper layers, 64.2 x 16.3 mm, 252 parts, among them J1 Conn_Coaxial_Small, J2 Conn_Coaxial_Small, J5 Conn_Coaxial, J6 Conn_Coaxial_Small, T1 0900PC16J0042001E, T2 0900PC16J0042001E, T5 0900PC16J0042001E, U1 ESP32-C3, U19 ESP32-C3, U2 TLV75533PDQNR, U20 TLV75533PDQNR, U21 SX1281IMLTRT, U22 ESP32-C3, U23 TLV75533PDQNR, U24 SX1281IMLTRT, U25 ESP32-C3, U26 TLV75533PDQNR, U27 LR1121IMLTRT, U28 RFX2401C, U29 SKY13373-460LF, U3 LR1121IMLTRT, U4 RFX2401C, U5 SKY13373-460LF, U6 LR1121IMLTRT, U7 RFX2401C, U8 SKY13373-460LF, U9 TS2306A 240GF MSM 9_C2976675, X1 CJ17-400001010B20, X3 CJ17-400001010B20, X4 CJ17-400001010B20, X5 CJ17-400001010B20

Commit message: Rev 3.1 working state: zone refills, fab option names, ordered sets
Mono and Gemini PCB zone refills and priority renumbering, Lite-UFL J1
LCSC field, fabrication-toolkit archive names per revision, the dated
2026-08-06 production sets for Lite-UFL and Mono as the record of what
was ordered, competitor RX catalogue, stale export STEPs deleted. The
repo-specific .gitignore tail restores flashing/bringup notes and the
firmware handoff bundle to local-only, plus regenerable dumps.

Co-Authored-By: Claude Opus 5 (1M context) <noreply@anthropic.com>
Parts:
- removed AE3, AE4, AE6: 2450AT18A100E, OpenRX-Shared:ANT-SMD_L3.2-W1.6
- removed AE5: 47948-0001, OpenRX-Shared:ANT-SMD_47948-0001
- removed C100, C117, C120, C125, C144, C147, C154, C92, C95: 10uF, Capacitor_SMD:C_0402_1005Metric
- removed C101, C115, C116, C118, C121, C122, C123, C126, C141, C142, C145, C148, C149, C150, C152, C90, C91, C93, C96, C97, C98: 100nF, Capacitor_SMD:C_0201_0603Metric
- removed C102, C127: 1nF, Capacitor_SMD:C_0201_0603Metric
- removed C103, C128, C156: 470nF, Capacitor_SMD:C_0201_0603Metric
- removed C104, C105, C129, C130, C165, C166: 1.2pF, Capacitor_SMD:C_0201_0603Metric
- removed C106, C108, C111, C114, C119, C124, C131, C133, C136, C140, C146, C153, C161, C163, C164, C167, C89, C94, C99: 1uF, Capacitor_SMD:C_0201_0603Metric
- removed C107, C109, C110, C132, C134, C135, C162: 10nF, Capacitor_SMD:C_0201_0603Metric
- removed C112, C113, C137, C139, C87, C88: 15pF, Capacitor_SMD:C_0201_0603Metric
- removed C138, C159, C160: 47p, Capacitor_SMD:C_0201_0603Metric
- removed C143: 10pF, Capacitor_SMD:C_0201_0603Metric
- removed C151: 47pF, Capacitor_SMD:C_0201_0603Metric
- removed C155: 2.2nF, Capacitor_SMD:C_0201_0603Metric
- removed C157: 220pF, Capacitor_SMD:C_0201_0603Metric
- removed C158: 1n, Capacitor_SMD:C_0201_0603Metric
- removed D3, D4, D5: XL-1010RGBC-WS2812B, OpenRX-Shared:LED-SMD_4P-L1.0-W1.0-TL_XL-1010RGBC-WS2812B
- removed FL5, FL6, FL7: 2450FM07D0034T, OpenRX-Shared:FILTER-SMD_4P-L1.0-W0.5-L
- removed J5: Conn_Coaxial, Connector_Coaxial:U.FL_Hirose_U.FL-R-SMT-1_Vertical
- removed J6: Conn_Coaxial_Small, Connector_Coaxial:U.FL_Hirose_U.FL-R-SMT-1_Vertical
- removed L15, L19, L24: 24nH, Inductor_SMD:L_0201_0603Metric
- removed L16, L20, L26: 2.5nH, Inductor_SMD:L_0201_0603Metric
- removed L17, L21, L25: 2.0nH, Inductor_SMD:L_0201_0603Metric
- removed L18, L22: 15uH, Inductor_SMD:L_0805_2012Metric
- removed L23: 10uH, Inductor_SMD:L_0603_1608Metric
- removed L27: 47nH, Inductor_SMD:L_0402_1005Metric
- removed OSC3, OSC4: OW7EL89CENUNFAYLC-52M, OpenRX-Shared:OSC-SMD_4P-L2.0-W1.6-BL_TXC_7Z
- removed OSC5: OW7EL89CENUYO3YLC-32M, OpenRX-Shared:OSC-SMD_4P-L2.0-W1.6-BL_TXC_7Z
- removed R25, R26, R27, R28, R29, R30, R31, R32, R34, R35, R36, R37: 10k, Resistor_SMD:R_0201_0603Metric
- removed R33: 200, Resistor_SMD:R_0201_0603Metric
- removed R38: 220, Resistor_SMD:R_0201_0603Metric
- removed R39, R40: 100k, Resistor_SMD:R_0201_0603Metric
- removed T5: 0900PC16J0042001E, OpenRX-Shared:FILTER-SMD_10P-L2.0-W1.6-BL
- removed TP10, TP15, TP20: TX, OpenRX-Shared:SolderPad_1.2x2.0mm
- removed TP11, TP16, TP21: 5V, OpenRX-Shared:SolderPad_1.2x2.0mm
- removed TP12, TP17, TP22: GND, OpenRX-Shared:SolderPad_1.2x2.0mm
- removed TP13, TP18, TP23: BOOT, OpenRX-Shared:SolderPad_1.2x2.0mm
- removed TP14, TP19, TP9: RX, OpenRX-Shared:SolderPad_1.2x2.0mm
- removed U19, U22, U25: ESP32-C3, Package_DFN_QFN:QFN-32-1EP_5x5mm_P0.5mm_EP3.7x3.7mm
- removed U20, U23, U26: TLV75533PDQNR, OpenRX-Shared:X2SON-4_L1.0-W1.0-P0.65-TL-EP
- removed U21, U24: SX1281IMLTRT, OpenRX-Shared:QFN-24_L4.0-W4.0-P0.50-TL-EP2.6
- removed U27: LR1121IMLTRT, Package_DFN_QFN:QFN-32-1EP_5x5mm_P0.5mm_EP3.7x3.7mm
- removed U28: RFX2401C, OpenRX-Shared:QFN-16_L3.0-W3.0-P0.50-BL-EP1.7
- removed U29: SKY13373-460LF, OpenRX-Shared:QFN-12_EP_2x2_Pitch0.5mm
- removed X3, X4, X5: CJ17-400001010B20, OpenRX-Shared:CRYSTAL-SMD_4P-L1.6-W1.2-BL
- added AE1: 2450AT18A100E, OpenRX-Shared:ANT-SMD_L3.2-W1.6, B.Cu at (145.8, 114.3)
- added AE1: 2450AT18A100E, OpenRX-Shared:ANT-SMD_L3.2-W1.6, B.Cu at (161.8, 114.3)
- added AE1: 2450AT18A100E, OpenRX-Shared:ANT-SMD_L3.2-W1.6, B.Cu at (123.8, 105.5)
- added AE2: 47948-0001, OpenRX-Shared:ANT-SMD_47948-0001, F.Cu at (161.9, 108.2)
- added C1: 15pF, Capacitor_SMD:C_0201_0603Metric, F.Cu at (163.8, 113.7)
- added C1: 15pF, Capacitor_SMD:C_0201_0603Metric, F.Cu at (147.8, 113.7)
- added C1: 15pF, Capacitor_SMD:C_0201_0603Metric, B.Cu at (125.8, 105.3)
- added C10: 1uF, Capacitor_SMD:C_0201_0603Metric, B.Cu at (123.0, 113.8)
- added C10: 1uF, Capacitor_SMD:C_0201_0603Metric, B.Cu at (139.0, 107.0)
- added C10: 1uF, Capacitor_SMD:C_0201_0603Metric, B.Cu at (155.0, 107.0)
- added C11: 10uF, Capacitor_SMD:C_0402_1005Metric, F.Cu at (144.1, 110.8)
- added C11: 10uF, Capacitor_SMD:C_0402_1005Metric, F.Cu at (160.1, 110.8)
- added C11: 10uF, Capacitor_SMD:C_0402_1005Metric, F.Cu at (132.1, 112.9)
- added C12: 100nF, Capacitor_SMD:C_0201_0603Metric, F.Cu at (123.4, 109.8)
- added C12: 100nF, Capacitor_SMD:C_0201_0603Metric, B.Cu at (157.7, 107.4)
- added C12: 100nF, Capacitor_SMD:C_0201_0603Metric, B.Cu at (141.7, 107.4)
- added C13: 100nF, Capacitor_SMD:C_0201_0603Metric, F.Cu at (125.1, 114.7)
- added C13: 100nF, Capacitor_SMD:C_0201_0603Metric, B.Cu at (140.2, 112.8)
- added C13: 100nF, Capacitor_SMD:C_0201_0603Metric, B.Cu at (156.2, 112.8)
- added C14: 100nF, Capacitor_SMD:C_0201_0603Metric, B.Cu at (141.3, 113.3)
- added C14: 100nF, Capacitor_SMD:C_0201_0603Metric, B.Cu at (125.8, 110.9)
- added C14: 100nF, Capacitor_SMD:C_0201_0603Metric, B.Cu at (157.3, 113.3)
- added C15: 1uF, Capacitor_SMD:C_0201_0603Metric, B.Cu at (156.2, 107.9)
- added C15: 47pF, Capacitor_SMD:C_0201_0603Metric, B.Cu at (125.8, 110.2)
- added C15: 1uF, Capacitor_SMD:C_0201_0603Metric, B.Cu at (140.2, 107.9)
- added C16: 10uF, Capacitor_SMD:C_0402_1005Metric, F.Cu at (139.8, 107.5)
- added C16: 10uF, Capacitor_SMD:C_0402_1005Metric, F.Cu at (155.8, 107.5)
- added C16: 100nF, Capacitor_SMD:C_0201_0603Metric, B.Cu at (129.9, 113.7)
- added C17: 1uF, Capacitor_SMD:C_0201_0603Metric, B.Cu at (123.9, 112.5)
- added C17: 100nF, Capacitor_SMD:C_0201_0603Metric, B.Cu at (157.7, 112.3)
- added C17: 100nF, Capacitor_SMD:C_0201_0603Metric, B.Cu at (141.7, 112.3)
- added C18: 10uF, Capacitor_SMD:C_0402_1005Metric, B.Cu at (123.7, 111.7)
- added C19: 1nF, Capacitor_SMD:C_0201_0603Metric, B.Cu at (138.6, 112.5)
- added C19: 2.2nF, Capacitor_SMD:C_0201_0603Metric, B.Cu at (125.8, 109.5)
- added C19: 1nF, Capacitor_SMD:C_0201_0603Metric, B.Cu at (154.6, 112.5)
- added C2: 47p, Capacitor_SMD:C_0201_0603Metric, F.Cu at (124.8, 109.0)
- added C20: 470nF, Capacitor_SMD:C_0201_0603Metric, F.Cu at (127.8, 114.9)
- added C20: 470nF, Capacitor_SMD:C_0201_0603Metric, B.Cu at (157.3, 114.8)
- added C20: 470nF, Capacitor_SMD:C_0201_0603Metric, B.Cu at (141.3, 114.8)
- added C21: 1.2pF, Capacitor_SMD:C_0201_0603Metric, B.Cu at (160.3, 113.0)
- added C21: 220pF, Capacitor_SMD:C_0201_0603Metric, B.Cu at (129.8, 104.8)
- added C21: 1.2pF, Capacitor_SMD:C_0201_0603Metric, B.Cu at (144.3, 113.0)
- added C22: 1n, Capacitor_SMD:C_0201_0603Metric, F.Cu at (128.1, 103.0)
- added C22: 1.2pF, Capacitor_SMD:C_0201_0603Metric, B.Cu at (163.2, 113.0)
- added C22: 1.2pF, Capacitor_SMD:C_0201_0603Metric, B.Cu at (147.2, 113.0)
- added C23: 1uF, Capacitor_SMD:C_0201_0603Metric, F.Cu at (159.6, 107.2)
- added C23: 47p, Capacitor_SMD:C_0201_0603Metric, F.Cu at (129.4, 101.8)
- added C23: 1uF, Capacitor_SMD:C_0201_0603Metric, F.Cu at (143.6, 107.2)
- added C24: 10nF, Capacitor_SMD:C_0201_0603Metric, F.Cu at (147.4, 111.2)
- added C24: 10nF, Capacitor_SMD:C_0201_0603Metric, F.Cu at (163.4, 111.2)
- added C24: 47p, Capacitor_SMD:C_0201_0603Metric, F.Cu at (125.7, 104.5)
- added C25: 1uF, Capacitor_SMD:C_0201_0603Metric, F.Cu at (145.7, 111.5)
- added C25: 1uF, Capacitor_SMD:C_0201_0603Metric, F.Cu at (131.8, 108.8)
- added C25: 1uF, Capacitor_SMD:C_0201_0603Metric, F.Cu at (161.7, 111.5)
- added C26: 10nF, Capacitor_SMD:C_0201_0603Metric, F.Cu at (131.6, 107.8)
- added C26: 10nF, Capacitor_SMD:C_0201_0603Metric, B.Cu at (139.1, 111.2)
- added C26: 10nF, Capacitor_SMD:C_0201_0603Metric, B.Cu at (155.1, 111.2)
- added C27: 1uF, Capacitor_SMD:C_0201_0603Metric, B.Cu at (125.8, 112.0)
- added C27: 10nF, Capacitor_SMD:C_0201_0603Metric, B.Cu at (155.1, 110.5)
- added C27: 10nF, Capacitor_SMD:C_0201_0603Metric, B.Cu at (139.1, 110.5)
- added C28: 1uF, Capacitor_SMD:C_0201_0603Metric, B.Cu at (126.0, 114.7)
- added C28: 1uF, Capacitor_SMD:C_0201_0603Metric, B.Cu at (141.4, 109.7)
- added C28: 1uF, Capacitor_SMD:C_0201_0603Metric, B.Cu at (157.4, 109.7)
- added C29: 1.2pF, Capacitor_SMD:C_0201_0603Metric, B.Cu at (131.9, 105.8)
- added C3: 15pF, Capacitor_SMD:C_0201_0603Metric, F.Cu at (160.9, 112.5)
- added C3: 15pF, Capacitor_SMD:C_0201_0603Metric, F.Cu at (144.9, 112.5)
- added C3: 15pF, Capacitor_SMD:C_0201_0603Metric, B.Cu at (128.6, 105.5)
- added C30: 1.2pF, Capacitor_SMD:C_0201_0603Metric, B.Cu at (131.3, 103.8)
- added C31: 1uF, Capacitor_SMD:C_0201_0603Metric, B.Cu at (129.8, 104.0)
- added C4: 1uF, Capacitor_SMD:C_0201_0603Metric, F.Cu at (162.7, 111.9)
- added C4: 1uF, Capacitor_SMD:C_0201_0603Metric, F.Cu at (132.2, 107.8)
- added C4: 1uF, Capacitor_SMD:C_0201_0603Metric, F.Cu at (146.7, 111.9)
- added C5: 100nF, Capacitor_SMD:C_0201_0603Metric, F.Cu at (158.9, 107.2)
- added C5: 100nF, Capacitor_SMD:C_0201_0603Metric, F.Cu at (142.9, 107.2)
- added C5: 100nF, Capacitor_SMD:C_0201_0603Metric, B.Cu at (131.1, 112.8)
- added C6: 100nF, Capacitor_SMD:C_0201_0603Metric, F.Cu at (159.6, 110.0)
- added C6: 100nF, Capacitor_SMD:C_0201_0603Metric, F.Cu at (143.9, 110.0)
- added C6: 100nF, Capacitor_SMD:C_0201_0603Metric, B.Cu at (126.5, 112.2)
- added C7: 10pF, Capacitor_SMD:C_0201_0603Metric, F.Cu at (123.8, 110.5)
- added C8: 10uF, Capacitor_SMD:C_0402_1005Metric, F.Cu at (138.8, 107.5)
- added C8: 10uF, Capacitor_SMD:C_0402_1005Metric, F.Cu at (154.8, 107.5)
- added C8: 10uF, Capacitor_SMD:C_0402_1005Metric, B.Cu at (123.7, 115.0)
- added C9: 100nF, Capacitor_SMD:C_0201_0603Metric, F.Cu at (132.2, 111.2)
- added C9: 100nF, Capacitor_SMD:C_0201_0603Metric, F.Cu at (143.9, 112.3)
- added C9: 100nF, Capacitor_SMD:C_0201_0603Metric, F.Cu at (159.9, 112.3)
- added D1: XL-1010RGBC-WS2812B, OpenRX-Shared:LED-SMD_4P-L1.0-W1.0-TL_XL-1010RGBC-WS2812B, F.Cu at (141.2, 107.5)
- added D1: XL-1010RGBC-WS2812B, OpenRX-Shared:LED-SMD_4P-L1.0-W1.0-TL_XL-1010RGBC-WS2812B, F.Cu at (157.2, 107.5)
- added D1: XL-1010RGBC-WS2812B, OpenRX-Shared:LED-SMD_4P-L1.0-W1.0-TL_XL-1010RGBC-WS2812B, F.Cu at (123.5, 108.6)
- added FL1: 2450FM07D0034T, OpenRX-Shared:FILTER-SMD_4P-L1.0-W0.5-L, F.Cu at (157.6, 108.9)
- added FL1: 2450FM07D0034T, OpenRX-Shared:FILTER-SMD_4P-L1.0-W0.5-L, F.Cu at (130.3, 107.2)
- added FL1: 2450FM07D0034T, OpenRX-Shared:FILTER-SMD_4P-L1.0-W0.5-L, F.Cu at (141.6, 108.9)
- added G***: LOGO, OpenRX-Shared:expresslrs_logo, F.Cu at (124.4, 105.8)
- added J1: Conn_Coaxial_Small, Connector_Coaxial:U.FL_Hirose_U.FL-R-SMT-1_Vertical, F.Cu at (124.8, 102.0)
- added J1: Conn_Coaxial, Connector_Coaxial:U.FL_Hirose_U.FL-R-SMT-1_Vertical, F.Cu at (146.2, 108.7)
- added L1: 24nH, Inductor_SMD:L_0201_0603Metric, F.Cu at (147.8, 112.2)
- added L1: 24nH, Inductor_SMD:L_0201_0603Metric, F.Cu at (163.8, 112.2)
- added L1: 10uH, Inductor_SMD:L_0603_1608Metric, B.Cu at (128.2, 114.0)
- added L2: 2.5nH, Inductor_SMD:L_0201_0603Metric, B.Cu at (161.8, 113.0)
- added L2: 2.5nH, Inductor_SMD:L_0201_0603Metric, B.Cu at (145.8, 113.0)
- added L2: 24nH, Inductor_SMD:L_0201_0603Metric, B.Cu at (127.7, 104.2)
- added L3: 2.0nH, Inductor_SMD:L_0201_0603Metric, F.Cu at (159.9, 111.6)
- added L3: 2.0nH, Inductor_SMD:L_0201_0603Metric, F.Cu at (132.2, 109.8)
- added L3: 2.0nH, Inductor_SMD:L_0201_0603Metric, F.Cu at (143.9, 111.6)
- added L4: 15uH, Inductor_SMD:L_0805_2012Metric, B.Cu at (142.8, 114.1)
- added L4: 15uH, Inductor_SMD:L_0805_2012Metric, B.Cu at (158.8, 114.1)
- added L4: 2.5nH, Inductor_SMD:L_0201_0603Metric, B.Cu at (131.1, 104.8)
- added L5: 47nH, Inductor_SMD:L_0402_1005Metric, F.Cu at (125.5, 107.8)
- added OSC1: OW7EL89CENUYO3YLC-32M, OpenRX-Shared:OSC-SMD_4P-L2.0-W1.6-BL_TXC_7Z, F.Cu at (124.0, 112.9)
- added OSC1: OW7EL89CENUNFAYLC-52M, OpenRX-Shared:OSC-SMD_4P-L2.0-W1.6-BL_TXC_7Z, B.Cu at (139.6, 114.4)
- added OSC1: OW7EL89CENUNFAYLC-52M, OpenRX-Shared:OSC-SMD_4P-L2.0-W1.6-BL_TXC_7Z, B.Cu at (155.6, 114.4)
- added R1: 200, Resistor_SMD:R_0201_0603Metric, F.Cu at (125.3, 107.0)
- added R2: 10k, Resistor_SMD:R_0201_0603Metric, F.Cu at (139.4, 108.9)
- added R2: 10k, Resistor_SMD:R_0201_0603Metric, F.Cu at (155.4, 108.9)
- added R2: 10k, Resistor_SMD:R_0201_0603Metric, B.Cu at (124.1, 110.7)
- added R3: 10k, Resistor_SMD:R_0201_0603Metric, B.Cu at (123.9, 108.7)
- added R3: 10k, Resistor_SMD:R_0201_0603Metric, B.Cu at (157.3, 108.5)
- added R3: 10k, Resistor_SMD:R_0201_0603Metric, B.Cu at (141.3, 108.5)
- added R4: 10k, Resistor_SMD:R_0201_0603Metric, B.Cu at (130.6, 115.0)
- added R4: 10k, Resistor_SMD:R_0201_0603Metric, B.Cu at (140.9, 107.4)
- added R4: 10k, Resistor_SMD:R_0201_0603Metric, B.Cu at (156.9, 107.4)
- added R5: 10k, Resistor_SMD:R_0201_0603Metric, B.Cu at (126.0, 114.0)
- added R5: 10k, Resistor_SMD:R_0201_0603Metric, B.Cu at (141.4, 111.1)
- added R5: 10k, Resistor_SMD:R_0201_0603Metric, B.Cu at (157.4, 111.1)
- added R6: 220, Resistor_SMD:R_0201_0603Metric, F.Cu at (124.8, 110.8)
- added R7: 100k, Resistor_SMD:R_0201_0603Metric, F.Cu at (132.2, 106.3)
- added R8: 100k, Resistor_SMD:R_0201_0603Metric, F.Cu at (132.1, 101.8)
- added T1: 0900PC16J0042001E, OpenRX-Shared:FILTER-SMD_10P-L2.0-W1.6-BL, F.Cu at (127.5, 107.0)
- added TP1: RX, OpenRX-Shared:SolderPad_1.2x2.0mm, F.Cu at (123.8, 118.0)
- added TP1: RX, OpenRX-Shared:SolderPad_1.2x2.0mm, F.Cu at (139.3, 118.0)
- added TP1: RX, OpenRX-Shared:SolderPad_1.2x2.0mm, F.Cu at (155.3, 118.0)
- added TP2: TX, OpenRX-Shared:SolderPad_1.2x2.0mm, F.Cu at (141.9, 118.0)
- added TP2: TX, OpenRX-Shared:SolderPad_1.2x2.0mm, F.Cu at (126.4, 118.0)
- added TP2: TX, OpenRX-Shared:SolderPad_1.2x2.0mm, F.Cu at (157.9, 118.0)
- added TP3: 5V, OpenRX-Shared:SolderPad_1.2x2.0mm, F.Cu at (144.4, 118.0)
- added TP3: 5V, OpenRX-Shared:SolderPad_1.2x2.0mm, F.Cu at (128.9, 118.0)
- added TP3: 5V, OpenRX-Shared:SolderPad_1.2x2.0mm, F.Cu at (160.4, 118.0)
- added TP4: GND, OpenRX-Shared:SolderPad_1.2x2.0mm, F.Cu at (131.5, 118.0)
- added TP4: GND, OpenRX-Shared:SolderPad_1.2x2.0mm, F.Cu at (147.0, 118.0)
- added TP4: GND, OpenRX-Shared:SolderPad_1.2x2.0mm, F.Cu at (163.0, 118.0)
- added TP5: TestPoint, TestPoint:TestPoint_Pad_D1.5mm, F.Cu at (101.1, 102.3)
- added TP5: BOOT, OpenRX-Shared:SolderPad_1.2x2.0mm, F.Cu at (147.3, 115.0)
- added TP5: BOOT, OpenRX-Shared:SolderPad_1.2x2.0mm, F.Cu at (163.3, 115.0)
- added TP5: BOOT, OpenRX-Shared:SolderPad_1.2x2.0mm, B.Cu at (131.9, 115.0)
- added U1: ESP32-C3, Package_DFN_QFN:QFN-32-1EP_5x5mm_P0.5mm_EP3.7x3.7mm, B.Cu at (145.1, 109.5)
- added U1: ESP32-C3, Package_DFN_QFN:QFN-32-1EP_5x5mm_P0.5mm_EP3.7x3.7mm, B.Cu at (129.6, 109.3)
- added U1: ESP32-C3, Package_DFN_QFN:QFN-32-1EP_5x5mm_P0.5mm_EP3.7x3.7mm, B.Cu at (161.1, 109.5)
- added U2: TLV75533PDQNR, OpenRX-Shared:X2SON-4_L1.0-W1.0-P0.65-TL-EP, B.Cu at (139.1, 108.0)
- added U2: TLV75533PDQNR, OpenRX-Shared:X2SON-4_L1.0-W1.0-P0.65-TL-EP, B.Cu at (124.0, 113.7)
- added U2: TLV75533PDQNR, OpenRX-Shared:X2SON-4_L1.0-W1.0-P0.65-TL-EP, B.Cu at (155.1, 108.0)
- added U3: SX1281IMLTRT, OpenRX-Shared:QFN-24_L4.0-W4.0-P0.50-TL-EP2.6, F.Cu at (156.8, 112.0)
- added U3: LR1121IMLTRT, Package_DFN_QFN:QFN-32-1EP_5x5mm_P0.5mm_EP3.7x3.7mm, F.Cu at (128.3, 111.5)
- added U3: SX1281IMLTRT, OpenRX-Shared:QFN-24_L4.0-W4.0-P0.50-TL-EP2.6, F.Cu at (140.8, 112.0)
- added U4: RFX2401C, OpenRX-Shared:QFN-16_L3.0-W3.0-P0.50-BL-EP1.7, F.Cu at (130.7, 104.1)
- added U5: SKY13373-460LF, OpenRX-Shared:QFN-12_EP_2x2_Pitch0.5mm, F.Cu at (127.5, 104.5)
- added X1: CJ17-400001010B20, OpenRX-Shared:CRYSTAL-SMD_4P-L1.6-W1.2-BL, F.Cu at (162.3, 113.2)
- added X1: CJ17-400001010B20, OpenRX-Shared:CRYSTAL-SMD_4P-L1.6-W1.2-BL, F.Cu at (146.3, 113.2)
- added X1: CJ17-400001010B20, OpenRX-Shared:CRYSTAL-SMD_4P-L1.6-W1.2-BL, B.Cu at (127.2, 105.3)
Connections:
- C13 pad 2: /Clock/VTCXO -> +3V3
- OSC1 pad 4: /Clock/VTCXO -> +3V3
- U3 pad 3: /LR1121_A/VTCXO -> unconnected-(U3-VTCXO-Pad3)
- U6 pad 3: /Clock/VTCXO -> unconnected-(U6-VTCXO-Pad3)
Routing:
- net GND: track 97.9 -> 40.7 mm, vias 234 -> 346
- net /ESP32-C3/BOOT: track 14.8 -> 35.7 mm, vias 2 -> 3
- net +3V3: track 87.5 -> 98.8 mm
- net Net-(OSC1-VDD): track 6.98 -> 0.00 mm
- net /Clock/VTCXO: track 2.80 -> 0.00 mm
- net Net-(U1-U0TXD): track 69.6 -> 72.0 mm
- net Net-(U3-VREG): track 4.97 -> 4.33 mm
Other:
- board size 64.2 x 16.3 mm -> 64.2 x 17.3 mm
