File: OpenRX-Gemini/esp32c3_lr1121_gemini.kicad_sch (KiCad schematic)
At the start: 68 parts, among them T4 0900PC16J0042001E, T5 0900PC16J0042001E, U1 OW7EL89CENUYO3YLC-32M, U15 RFX2401C, U16 SKY13414-485LF, U17 RFX2401C, U18 SKY13414-485LF, U2 LR1121IMLTRT, U3 ESP32-C3FH4, U4 TS2306A 240GF MSM 9_C2976675, U6 TLV75533PDQNR, U9 LR1121IMLTRT, X1 CJ17-400001010B20

Commit message: sch: standardise LCSC/Manufacturer/MPN fields across all variants
Migrated LCSC part numbers out of variant-specific LCSC_Part fields into
the standard LCSC field, and backfilled Manufacturer/MPN from the LCSC
catalogue, on all four board variants (Gemini, Lite, Lite-UFL, Mono) and
the shared ESP32-C3/SX1281 RX core sheet.

kicad-skip reflowed each file on save, so the diffs are large but purely
formatting; a structural S-expression diff and ERC re-run on all 12
affected schematics (including the 4 unmodified top-level sheets) confirm
only property values changed, no nets/placement/footprints touched.

Known gap: L2/L3 in OpenRX-Gemini/esp32c3_lr1121_gemini.kicad_sch carry
LCSC C1035, which no longer resolves in the LCSC catalogue, so they have
no Manufacturer/MPN. Universal BOM lines for those parts will be
incomplete until a replacement part is sourced.

Co-Authored-By: Claude Fable 5 <noreply@anthropic.com>
Parts:
- AE1: MPN (none) -> 2450AT18A100E; Manufacturer (none) -> Johanson Dielectrics
- C1, C4: MPN (none) -> 0201CG180J500NT; Manufacturer (none) -> FH
- C10, C11, C12, C13, C15, C17, C18, C24, C25, C26, C29, C3, C7: MPN (none) -> GRM033R61E104KE14D; Manufacturer (none) -> muRata
- C14, C22: MPN (none) -> CL05A106MQ5NUNC; Manufacturer (none) -> Samsung Electro-Mechanics
- C16, C2, C20, C44, C47, C6: MPN (none) -> GRM033R61A105ME44D; Manufacturer (none) -> muRata
- C27, C8: MPN (none) -> GRM0335C1H100JA01D; Manufacturer (none) -> muRata
- C28, C9: MPN (none) -> CL05A475MP5NRNC; Manufacturer (none) -> Samsung Electro-Mechanics
- C42, C45: MPN (none) -> GRM0335C1HR30BA01D; Manufacturer (none) -> muRata
- C43, C46: MPN (none) -> 0201B221K500NT; Manufacturer (none) -> FH
- D1: MPN (none) -> XL-1010RGBC-2812B; Manufacturer (none) -> XINGLIGHT
- FL4, FL5: LCSC (none) -> C2651081; LCSC Part C2651081 -> (none)
- JP4, JP5: MPN (none) -> U.FL-R-SMT-1(80); Manufacturer (none) -> HRS
- L1: MPN (none) -> LQP03TN24NH02D; Manufacturer (none) -> muRata
- R1, R11, R2, R4, R5, R6, R7: MPN (none) -> RC0201FR-0710KL; Manufacturer (none) -> YAGEO
- R10, R9: MPN (none) -> RC0201FR-07680RL; Manufacturer (none) -> YAGEO
- R3, R8: MPN (none) -> RC0201FR-07220RL; Manufacturer (none) -> YAGEO
- T4, T5: MPN (none) -> 0900PC16J0042001E; Manufacturer (none) -> Johanson Dielectrics
- U1: MPN (none) -> OW7EL89CENUYO3YLC-32M; Manufacturer (none) -> YXC Crystal Oscillators
- U15, U17: MPN (none) -> RFX2401C; Manufacturer (none) -> SKYWORKS
- U16, U18: LCSC (none) -> C255353; LCSC Part C255353 -> (none)
- U2, U9: MPN (none) -> LR1121IMLTRT; Manufacturer (none) -> SEMTECH
- U3: MPN (none) -> ESP32-C3FH4; Manufacturer (none) -> ESPRESSIF
- U4: MPN (none) -> TS2306A 240gf MSM 9; Manufacturer (none) -> SHOU HAN
- U6: MPN (none) -> TLV75533PDQNR; Manufacturer (none) -> TI
- X1: MPN (none) -> CJ17-400001010B20; Manufacturer (none) -> JSCJ
