File: OpenRX-Lite-UFL/OpenRX-Lite-UFL.kicad_pcb (KiCad board)
At the start: 6 copper layers, 10 x 10.5 mm, 47 parts, among them J1 Conn_Coaxial, U1 ESP32-C3, U2 TLV75533PDQNR, U3 SX1281IMLTRT, X1 CJ17-400001010B20

Commit message: changed 3.3V supply on clocks, added text, enlarged pads
Parts:
- moved TP1 1.00 mm to (101.2, 111.0)
- moved TP2 1.00 mm to (103.7, 111.0)
- moved TP3 1.00 mm to (106.3, 111.0)
- moved TP4 1.00 mm to (108.8, 111.0)
Routing:
- net Net-(U1-U0TXD): track 10.1 -> 11.1 mm
Other:
- board size 10 x 10.5 mm -> 10 x 11.5 mm
