File: OpenRX-Lite-UFL/esp32c3_sx1281_lite.kicad_sch (KiCad schematic)
At the start: 47 parts, among them J1 Conn_Coaxial, U1 ESP32-C3, U2 TLV75533PDQNR, U3 SX1281IMLTRT, X1 CJ17-400001010B20

Commit message: Rev 3.1 working state: zone refills, fab option names, ordered sets
Mono and Gemini PCB zone refills and priority renumbering, Lite-UFL J1
LCSC field, fabrication-toolkit archive names per revision, the dated
2026-08-06 production sets for Lite-UFL and Mono as the record of what
was ordered, competitor RX catalogue, stale export STEPs deleted. The
repo-specific .gitignore tail restores flashing/bringup notes and the
firmware handoff bundle to local-only, plus regenerable dumps.

Co-Authored-By: Claude Opus 5 (1M context) <noreply@anthropic.com>
Parts:
- J1: LCSC (none) -> C88374
Changed lines of the file:
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@@
+			)
+		)
+		(property "LCSC" " C88374"
+			(at 187.96 116.84 0)
+			(hide yes)
+			(show_name no)
+			(do_not_autoplace no)
+			(effects
+				(font
+					(size 1.27 1.27)
+				)
 			)
 		)

Commit message: Lite-UFL J1: LCSC C88374, no leading space, on board and schematic
The schematic had ' C88374' with a leading space and the board had no
LCSC field at all, so the U.FL connector silently dropped out of the
fab BOM: check_export.py C3 caught it (bom 0 < sch 1). Schematic fixed
by one-string replacement; board field added via the pcbnew API, styled
like every other hidden LCSC field. Export re-run and verified.

Co-Authored-By: Claude Opus 5 (1M context) <noreply@anthropic.com>
Parts:
- J1: LCSC C88374 -> C88374
Changed lines of the file:
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@@
 			)
 		)
-		(property "LCSC" " C88374"
+		(property "LCSC" "C88374"
 			(at 187.96 116.84 0)
 			(hide yes)

Commit message: sch: standardise LCSC/Manufacturer/MPN fields across all variants
Migrated LCSC part numbers out of variant-specific LCSC_Part fields into
the standard LCSC field, and backfilled Manufacturer/MPN from the LCSC
catalogue, on all four board variants (Gemini, Lite, Lite-UFL, Mono) and
the shared ESP32-C3/SX1281 RX core sheet.

kicad-skip reflowed each file on save, so the diffs are large but purely
formatting; a structural S-expression diff and ERC re-run on all 12
affected schematics (including the 4 unmodified top-level sheets) confirm
only property values changed, no nets/placement/footprints touched.

Known gap: L2/L3 in OpenRX-Gemini/esp32c3_lr1121_gemini.kicad_sch carry
LCSC C1035, which no longer resolves in the LCSC catalogue, so they have
no Manufacturer/MPN. Universal BOM lines for those parts will be
incomplete until a replacement part is sourced.

Co-Authored-By: Claude Fable 5 <noreply@anthropic.com>
Parts:
- AE1: MPN (none) -> 2450AT18A100E; Manufacturer (none) -> Johanson Dielectrics
- C1, C3: MPN (none) -> GRM0335C1H150JA01D; Manufacturer (none) -> muRata
- C10, C15, C23, C25, C28, C4: MPN (none) -> GRM033R61A105ME44D; Manufacturer (none) -> muRata
- C11: MPN (none) -> GRM155R60J106ME44D; Manufacturer (none) -> muRata
- C12, C13, C14, C17, C5, C6, C9: MPN (none) -> GRM033R61E104KE14D; Manufacturer (none) -> muRata
- C16, C8: MPN (none) -> CL05A106MQ5NUNC; Manufacturer (none) -> Samsung Electro-Mechanics
- C19: MPN (none) -> 0201B102K500NT; Manufacturer (none) -> FH
- C20: MPN (none) -> GRM033R60J474KE90D; Manufacturer (none) -> muRata
- C21, C22: MPN (none) -> GRM0335C1H1R2BA01D; Manufacturer (none) -> muRata
- C24, C26, C27: MPN (none) -> GRM033R61A103KA01J; Manufacturer (none) -> muRata
- D1: LCSC (none) -> C5349953; LCSC Part C5349953 -> (none); MPN (none) -> XL-1010RGBC-2812B; Manufacturer (none) -> XINGLIGHT
- FL1: LCSC (none) -> C2651081; LCSC Part C2651081 -> (none)
- J1: MPN (none) -> U.FL-R-SMT-1(80); Manufacturer (none) -> HRS
- L1: MPN (none) -> LQP03TN24NH02D; Manufacturer (none) -> muRata
- L2: MPN (none) -> LQP03TN2N5C02D; Manufacturer (none) -> muRata
- L3: MPN (none) -> LQP03TN2N0B02D; Manufacturer (none) -> muRata
- OSC1: MPN (none) -> OW7EL89CENUNFAYLC-52M; Manufacturer (none) -> YXC Crystal Oscillators
- R2, R3, R4, R5: MPN (none) -> RC0201FR-0710KL; Manufacturer (none) -> YAGEO
- U2: MPN (none) -> TLV75533PDQNR; Manufacturer (none) -> TI
- U3: MPN (none) -> SX1281IMLTRT; Manufacturer (none) -> SEMTECH
- X1: MPN (none) -> CJ17-400001010B20; Manufacturer (none) -> JSCJ
