File: shared/sheets/esp32c3_sx1281_rx_core.kicad_sch (KiCad schematic)
At the start: 40 parts, among them U1 ESP32-C3FH4, U2 TLV75533PDQNR, U3 SX1281IMLTRT, U4 RFX2401C, X1 CJ17-400001010B20

Commit message: sch: standardise LCSC/Manufacturer/MPN fields across all variants
Migrated LCSC part numbers out of variant-specific LCSC_Part fields into
the standard LCSC field, and backfilled Manufacturer/MPN from the LCSC
catalogue, on all four board variants (Gemini, Lite, Lite-UFL, Mono) and
the shared ESP32-C3/SX1281 RX core sheet.

kicad-skip reflowed each file on save, so the diffs are large but purely
formatting; a structural S-expression diff and ERC re-run on all 12
affected schematics (including the 4 unmodified top-level sheets) confirm
only property values changed, no nets/placement/footprints touched.

Known gap: L2/L3 in OpenRX-Gemini/esp32c3_lr1121_gemini.kicad_sch carry
LCSC C1035, which no longer resolves in the LCSC catalogue, so they have
no Manufacturer/MPN. Universal BOM lines for those parts will be
incomplete until a replacement part is sourced.

Co-Authored-By: Claude Fable 5 <noreply@anthropic.com>
Parts:
- AE1: LCSC (none) -> C89334; LCSC Part C89334 -> (none); MPN (none) -> 2450AT18A100E; Manufacturer (none) -> Johanson Dielectrics
- C1, C13, C14, C15, C17, C2, C3, C4, C5: MPN (none) -> GRM033R61E104KE14D; Manufacturer (none) -> muRata
- C10, C19, C21, C8, C9: MPN (none) -> GRM033R61A105ME44D; Manufacturer (none) -> muRata
- C11, C12: MPN (none) -> CL05A106MQ5NUNC; Manufacturer (none) -> Samsung Electro-Mechanics
- C16: MPN (none) -> GRM033R60J474KE90D; Manufacturer (none) -> muRata
- C18: MPN (none) -> 0201B102K500NT; Manufacturer (none) -> FH
- C6, C7: MPN (none) -> CGA0201C0G100J500ET; Manufacturer (none) -> HRE
- D1: LCSC (none) -> C5349953; LCSC Part C5349953 -> (none); MPN (none) -> XL-1010RGBC-2812B; Manufacturer (none) -> XINGLIGHT
- JP1: LCSC (none) -> C88374; LCSC Part C88374 -> (none); MPN (none) -> U.FL-R-SMT-1(80); Manufacturer (none) -> HRS
- OSC1: LCSC (none) -> C22434896; LCSC Part C22434896 -> (none); MPN (none) -> OW7EL89CENUNFAYLC-52M; Manufacturer (none) -> YXC Crystal Oscillators
- R1, R2, R3, R4: MPN (none) -> RC0201FR-0710KL; Manufacturer (none) -> YAGEO
- U1: LCSC (none) -> C2858491; LCSC Part C2858491 -> (none); MPN (none) -> ESP32-C3FH4; Manufacturer (none) -> ESPRESSIF
- U2: LCSC (none) -> C2861882; LCSC Part C2861882 -> (none); MPN (none) -> TLV75533PDQNR; Manufacturer (none) -> TI
- U3: LCSC (none) -> C2151551; LCSC Part C2151551 -> (none); MPN (none) -> SX1281IMLTRT; Manufacturer (none) -> SEMTECH
- U4: LCSC (none) -> C19213; LCSC Part C19213 -> (none); MPN (none) -> RFX2401C; Manufacturer (none) -> SKYWORKS
- USB1: LCSC (none) -> C574024; LCSC Part C574024 -> (none); MPN (none) -> DEA102700LT-6307A2; Manufacturer (none) -> TDK
- X1: LCSC (none) -> C2875272; LCSC Part C2875272 -> (none); MPN (none) -> CJ17-400001010B20; Manufacturer (none) -> JSCJ
